File: watering/watering.kicad_sch (KiCad schematic)
At the start: 20 parts, among them J1 Screw_Terminal_01x02, J2 Screw_Terminal_01x03, J3 Screw_Terminal_01x02, J4 Screw_Terminal_01x02, J5 Screw_Terminal_01x03, J6 Screw_Terminal_01x02, J7 Screw_Terminal_01x02

Commit message: Update to KiCAD v9.0
Parts:
- A1: footprint watering:Tiny2040 -> watering:TINY2040
Changed lines of the file:
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@@
 (kicad_sch
-	(version 20231120)
+	(version 20250114)
 	(generator "eeschema")
-	(generator_version "8.0")
+	(generator_version "9.0")
 	(paper "A4")
 	(title_block
@@
 			)
 		)
-		(property "Footprint" "watering:Tiny2040"
+		(property "Footprint" "watering:TINY2040"
 			(at 99.06 69.85 0)
 			(effects
@@
 		)
 	)
+	(embedded_fonts no)
 )
